File: doorbell/doorbell.kicad_pcb (KiCad board)
At the start: 2 copper layers, 0 parts

Commit message: Updating schematic to be multiple sheets, including gerber files for PCB, updating readme
Parts:
- added C201: 470u, Capacitor_THT:CP_Radial_D10.0mm_P5.00mm, F.Cu at (150.5, 120.5)
- added C202: 330uF, Capacitor_THT:CP_Radial_D10.0mm_P5.00mm, F.Cu at (150.5, 135.0)
- added C301: 10uF, Capacitor_THT:C_Disc_D5.0mm_W2.5mm_P5.00mm, F.Cu at (172.0, 55.5)
- added C302: 0.01uF, Capacitor_THT:C_Disc_D5.0mm_W2.5mm_P5.00mm, F.Cu at (178.5, 83.0)
- added C303: 10uF, Capacitor_THT:C_Disc_D5.0mm_W2.5mm_P5.00mm, F.Cu at (188.0, 78.5)
- added C401: 10uF, Capacitor_THT:C_Disc_D5.0mm_W2.5mm_P5.00mm, F.Cu at (132.0, 71.5)
- added C402: 0.01uF, Capacitor_THT:C_Disc_D5.0mm_W2.5mm_P5.00mm, F.Cu at (133.5, 93.0)
- added C403: 10uF, Capacitor_THT:C_Disc_D5.0mm_W2.5mm_P5.00mm, F.Cu at (139.5, 80.5)
- added C501: 10uF, Capacitor_THT:C_Disc_D5.0mm_W2.5mm_P5.00mm, F.Cu at (131.5, 122.5)
- added C502: 0.01uF, Capacitor_THT:C_Disc_D5.0mm_W2.5mm_P5.00mm, F.Cu at (144.0, 138.0)
- added C503: 10uF, Capacitor_THT:C_Disc_D5.0mm_W2.5mm_P5.00mm, F.Cu at (137.0, 136.5)
- added D201: 1N4002, Diode_THT:D_DO-41_SOD81_P10.16mm_Horizontal, F.Cu at (161.9, 100.5)
- added D202: 1N4002, Diode_THT:D_DO-41_SOD81_P10.16mm_Horizontal, F.Cu at (156.5, 110.7)
- added D203: 1N4002, Diode_THT:D_DO-41_SOD81_P10.16mm_Horizontal, F.Cu at (176.5, 110.7)
- added D204: 1N4002, Diode_THT:D_DO-41_SOD81_P10.16mm_Horizontal, F.Cu at (161.9, 110.5)
- added D205: 1N5817, Diode_THT:D_DO-41_SOD81_P10.16mm_Horizontal, F.Cu at (159.8, 129.5)
- added D301: 1N5817, Diode_THT:D_DO-41_SOD81_P10.16mm_Horizontal, F.Cu at (182.0, 64.2)
- added D302: 1N5817, Diode_THT:D_DO-41_SOD81_P10.16mm_Horizontal, F.Cu at (164.8, 82.0)
- added D303: 1N5817, Diode_THT:D_DO-41_SOD81_P10.16mm_Horizontal, F.Cu at (164.8, 89.0)
- added D401: 1N5817, Diode_THT:D_DO-41_SOD81_P10.16mm_Horizontal, F.Cu at (142.5, 75.7)
- added D402: 1N5817, Diode_THT:D_DO-41_SOD81_P10.16mm_Horizontal, F.Cu at (119.3, 92.5)
- added D403: 1N5817, Diode_THT:D_DO-41_SOD81_P10.16mm_Horizontal, F.Cu at (119.3, 96.8)
- added D501: 1N5817, Diode_THT:D_DO-41_SOD81_P10.16mm_Horizontal, F.Cu at (143.0, 127.7)
- added D502: 1N5817, Diode_THT:D_DO-41_SOD81_P10.16mm_Horizontal, F.Cu at (114.8, 142.5)
- added D503: 1N5817, Diode_THT:D_DO-41_SOD81_P10.16mm_Horizontal, F.Cu at (130.8, 144.0)
- added J101: 1-284392-2, Connector_TE-Connectivity:SHDR12W100P0X381_1X12_4572X820X1280P, F.Cu at (103.0, 45.7)
- added K302: G6E, Relay_THT:Relay_SPDT_Omron_G6E, F.Cu at (160.8, 82.2)
- added K402: G6E, Relay_THT:Relay_SPDT_Omron_G6E, F.Cu at (112.8, 93.2)
- added K502: G6E, Relay_THT:Relay_SPDT_Omron_G6E, F.Cu at (110.5, 143.7)
- added L201: 330uH, Inductor_THT:L_Toroid_Vertical_L24.6mm_W15.5mm_P11.44mm_Pulse_KM-4, F.Cu at (187.0, 128.0)
- added R301: 6k, Resistor_THT:R_Axial_DIN0411_L9.9mm_D3.6mm_P15.24mm_Horizontal, F.Cu at (153.0, 63.4)
- added R302: 10k, Resistor_THT:R_Axial_DIN0207_L6.3mm_D2.5mm_P10.16mm_Horizontal, F.Cu at (189.0, 64.2)
- added R303: 1k, Resistor_THT:R_Axial_DIN0207_L6.3mm_D2.5mm_P10.16mm_Horizontal, F.Cu at (177.0, 64.1)
- added R304: 10k, Resistor_THT:R_Axial_DIN0207_L6.3mm_D2.5mm_P10.16mm_Horizontal, F.Cu at (180.0, 78.1)
- added R401: 6k, Resistor_THT:R_Axial_DIN0411_L9.9mm_D3.6mm_P15.24mm_Horizontal, F.Cu at (112.8, 74.5)
- added R402: 10k, Resistor_THT:R_Axial_DIN0207_L6.3mm_D2.5mm_P10.16mm_Horizontal, F.Cu at (145.0, 52.0)
- added R403: 1k, Resistor_THT:R_Axial_DIN0207_L6.3mm_D2.5mm_P10.16mm_Horizontal, F.Cu at (137.5, 75.6)
- added R404: 10k, Resistor_THT:R_Axial_DIN0207_L6.3mm_D2.5mm_P10.16mm_Horizontal, F.Cu at (132.5, 88.7)
- added R501: 6k, Resistor_THT:R_Axial_DIN0411_L9.9mm_D3.6mm_P15.24mm_Horizontal, F.Cu at (111.3, 125.5)
- added R502: 10k, Resistor_THT:R_Axial_DIN0207_L6.3mm_D2.5mm_P10.16mm_Horizontal, F.Cu at (142.5, 114.2)
- added R503: 1k, Resistor_THT:R_Axial_DIN0207_L6.3mm_D2.5mm_P10.16mm_Horizontal, F.Cu at (138.0, 127.2)
- added R504: 10k, Resistor_THT:R_Axial_DIN0207_L6.3mm_D2.5mm_P10.16mm_Horizontal, F.Cu at (130.5, 140.2)
- added RV301: 10k, Potentiometer_THT:Potentiometer_Vishay_T93YA_Vertical, F.Cu at (186.0, 49.1)
- added RV302: 100k, Potentiometer_THT:Potentiometer_Vishay_T73YP_Vertical, F.Cu at (188.0, 74.1)
- added RV401: 10k, Potentiometer_THT:Potentiometer_Vishay_T93YA_Vertical, F.Cu at (107.0, 54.5)
- added RV402: 100k, Potentiometer_THT:Potentiometer_Vishay_T73YP_Vertical, F.Cu at (107.0, 70.0)
- added RV501: 10k, Potentiometer_THT:Potentiometer_Vishay_T93YA_Vertical, F.Cu at (105.5, 105.0)
- added RV502: 100k, Potentiometer_THT:Potentiometer_Vishay_T73YP_Vertical, F.Cu at (105.5, 121.5)
- added T301: CT05-1000, Transformer_THT:CT051000, F.Cu at (166.6, 57.9)
- added T401: CT05-1000, Transformer_THT:CT051000, F.Cu at (126.0, 69.0)
- added T501: CT05-1000, Transformer_THT:CT051000, F.Cu at (125.5, 120.0)
- added U201: LM2575-12WT, Package_TO_SOT_THT:TO-262-5_Vertical, F.Cu at (161.9, 122.0)
- added U301: LM358, Package_DIP:DIP-8_W7.62mm, F.Cu at (172.2, 42.7)
- added U302: COM-16473 (NA555), Package_DIP:DIP-8_W7.62mm, F.Cu at (173.5, 69.0)
- added U401: LM358, Package_DIP:DIP-8_W7.62mm, F.Cu at (131.5, 53.5)
- added U402: COM-16473 (NA555), Package_DIP:DIP-8_W7.62mm, F.Cu at (126.8, 79.7)
- added U501: LM358, Package_DIP:DIP-8_W7.62mm, F.Cu at (130.5, 104.5)
- added U502: COM-16473 (NA555), Package_DIP:DIP-8_W7.62mm, F.Cu at (123.5, 130.5)
Routing:
- net /current_sense_relay_1/GND: track 0.00 -> 490.3 mm, vias 0 -> 2
- net /current_sense_relay_1/12V: track 0.00 -> 405.0 mm
- net /transformer_1: track 0.00 -> 232.3 mm
- net /chime_common: track 0.00 -> 194.0 mm
- net /transformer_2: track 0.00 -> 174.7 mm
- net /chime_3: track 0.00 -> 134.2 mm
- net /button_3: track 0.00 -> 112.9 mm
- net /chime_2: track 0.00 -> 81.7 mm, vias 0 -> 2
- net Net-(D301-A): track 0.00 -> 54.7 mm
- net Net-(D401-K): track 0.00 -> 53.3 mm
- net Net-(U402-DIS): track 0.00 -> 49.1 mm
- net Net-(U502-DIS): track 0.00 -> 48.5 mm
- net /chime_1: track 0.00 -> 44.2 mm
- net Net-(D501-K): track 0.00 -> 43.5 mm
- net /button_1: track 0.00 -> 40.9 mm
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Other:
- board outline added: 98 x 112.5 mm
- net class Default removed
- board text added: "C1"
- board text added: "C2"
- board text added: "C3"
- board text added: "CC"
- board text added: "DB1"
- board text added: "DB1 Ring Duration"
- board text added: "DB1 Sensitivity"
- board text added: "DB2"
- board text added: "DB2 Ring Duration"
- board text added: "DB2 Sensitivity"
- board text added: "DB3"
- board text added: "DB3 Ring Duration"
- board text added: "DB3 Sensitivity"
- board text added: "Matt Stanford"
- board text added: "Video Doorbell Adapter"
- board text added: "trans"
- board text added: "v0.1"
